File: KiCAD-Project/JACC64-512K.kicad_sch (KiCad schematic)
At the start: 15 parts, among them SW1 SW_Push, SW2 SW_DIP_x05, U2 SST39SF040

Commit message: Added PDF schematics
Other:
- company: (none) -> Oddsocks b5s4
- title: (none) -> JACC64-512K
Changed lines of the file:
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@@
 	(generator_version "9.0")
 	(paper "A3")
+	(title_block
+		(title "JACC64-512K")
+		(rev "1.1")
+		(company "Oddsocks b5s4")
+	)
 	(junction
 		(at 274.32 138.43)
@@
 		(at 199.39 191.77)
 		(diameter 0)
-		(color 0 0 0 0)
+		(color 0 0 0 1)
 	)
 	(junction
@@
 		(at 199.39 181.61)
 		(diameter 0)
-		(color 0 0 0 0)
+		(color 0 0 0 1)
 	)
 	(junction
@@
 		(at 162.56 77.47)
 		(diameter 0)
-		(color 0 0 0 0)
+		(color 255 0 0 1)
 	)
 	(junction
@@
 		(at 129.54 163.83)
 		(diameter 0)
-		(color 0 0 0 0)
+		(color 255 153 0 1)
 	)
 	(no_connect
